Commit message: 调整特权信息、腿部动作低层实现（论文手动计算力矩，为了方便后面替换为执行器网络，本地使用DCmotor计算力矩）

File: source/robot_lab/data/Robots/unitree/go2arm_description/urdf/go2_piper_description_mjc_NoGripper.urdf (robot description, URDF)
Before this commit: robot go2arm_description, 49 links, 48 joints
Joints:
- joint base_mount_joint: origin xyz=0 0 0.072 rpy=0 0 0 -> xyz=0.10 0 0.072 rpy=0 0 0

Commit message: 修改urdf(机械臂安装位置)和机械臂PD，加了机械臂是否真冻结的debug检测

File: source/robot_lab/data/Robots/unitree/go2arm_description/urdf/go2_piper_description_mjc_NoGripper.urdf (robot description, URDF)
Before this commit: robot go2arm_description, 49 links, 48 joints
Joints:
- joint arm_mount_joint: origin xyz=0 0 0.015 rpy=0 0 0 -> xyz=0 0 0 rpy=0 0 0
- joint base_mount_joint: origin xyz=0.10 0 0.072 rpy=0 0 0 -> xyz=-0.01 0 0.085 rpy=0 0 0
